File: mixer.brd (EAGLE design)
At the start: 190 x 190 mm, 319 parts, among them U1 TL074IDT, U2 TL074IDT, U3 TL074IDT, U4 TL074IDT, U5 TL074IDT, U6 TL074IDT, U7 TL074IDT

Commit message: Started board layout and removed EQ
Parts:
- removed C39, CH1:C13, CH1:C14, CH1:C15, CH1:C16, CH1:C18, CH1:C20, CH2:C13, CH2:C14, CH2:C15, CH2:C16, CH2:C18, CH2:C20, CH3:C13, CH3:C14, CH3:C15, CH3:C16, CH3:C18, CH3:C20: 10u, 16V, passives:SV-A
- removed C40, C41, C42: 100 n, passives:C0603
- removed CH1:BLEND1, CH2:BLEND1, CH3:BLEND1: 50 k, passives:RK09L124000Z
- removed CH1:FR1, CH1:FR2, CH1:FRQ1, CH1:FRQ2, CH1:Q1, CH1:Q2, CH2:FR1, CH2:FR2, CH2:FRQ1, CH2:FRQ2, CH2:Q1, CH2:Q2, CH3:FR1, CH3:FR2, CH3:FRQ1, CH3:FRQ2, CH3:Q1, CH3:Q2, GAIN: 10 k, passives:RK09L1140
- removed CH1:R1, CH1:R7, CH2:R1, CH2:R7, CH3:R1, CH3:R7: 2.7 k, passives:R0603
- removed CH1:R2, CH1:R4, CH2:R2, CH2:R4, CH3:R2, CH3:R4: 470 k, passives:R0603
- removed CH1:R3, CH1:R6, CH2:R3, CH2:R6, CH3:R3, CH3:R6: 51 k, passives:R0603
- removed CH1:R5, CH2:R5, CH3:R5: 10 k, passives:R0603
- removed CH1:TC, CH2:TC, CH3:TC, TC, TC1, TC2, TC3: HOT_COLD, connectors:HOT_COLD
- removed CH1:U$1, CH2:U$1, CH3:U$1, U$2: SEND_RETURN, connectors:STEREO_TELE
- removed CH1:U$2, CH2:U$2, CH3:U$2: RK09L1140, passives:RK09L1140
- removed U$3, U$4: LEFT_RIGHT, connectors:LEFT_RIGHT
- added BYPASS, MONO: BUTTON, connectors:3-HOLES
- added CH1:BLEND, CH2:BLEND, CH3:BLEND: 50 k, passives:RK09L124000Z
- added CH1:IN, CH2:IN, CH3:IN, MON_IN, MON_THROUGH, OUT_L, OUT_R, TC_SEND_JACK: HOT_COLD, connectors:HOT_COLD
- added CH1:LEVEL, CH2:LEVEL, CH3:LEVEL: RK09L1140, passives:RK09L1140
- added D1, D2: 1N4004, passives:DO41-10
- added GAIN5: 10 k, passives:RJ9W
- added LD1: (no value), passives:DUOLED-A-5MM
- added LOOPMASTER: SEND_RETURN, connectors:SND_RET
- added MON_OUT: LEFT_RIGHT, connectors:LEFT_RIGHT
- added R64, R65: 10 k, passives:0204/7
- added TC_RET: LEFT_RIGHT_BYPASS, connectors:LEFT_RIGHT_BYPASS
- added U$10: SBC1-102-211, passives:SBC1-102-211
- added U$5: ADG333ABNZADG333ABNZ, ic:DIP762W53P254L2591H508Q20B
- added U$6: ADG436BNZADG436BNZ, ic:DIP762W53P254L2006H508Q16B
- added U8: TL074, ic:DIP762W53P254L1969H508Q14B
- added U9: V7809W-500R, power:CONV_V7809W-500R
- C1, C10, C13, C14, C15, C16, C18, C2, C20, C22, C3, C36, C4, C5, C8, C9, CH1:C12, CH1:C8, CH1:C9, CH2:C12, CH2:C8, CH2:C9, CH3:C12, CH3:C8, CH3:C9: value 10u, 16V -> 10u; device passives:SV-A -> passives:E2,0-5
- C11, C26, CH1:C10, CH2:C10, CH3:C10: value 100 n -> 10u; device passives:C0603 -> passives:E2,0-5
- C12, C21, C24, C25, C32, C6, C7: value 33u, 63V -> 10u, 63V; device passives:SV-E/F -> passives:E2,0-6
- C17, C19, C28, C29, C34, C35, C37, C38, CH1:C11, CH1:C17, CH1:C19, CH1:C4, CH2:C11, CH2:C17, CH2:C19, CH2:C4, CH3:C11, CH3:C17, CH3:C19, CH3:C4: device passives:C0603 -> passives:C025-025X050
- C23: value 10u, 16V -> 10u, 63V; device passives:SV-A -> passives:E2,0-6
- C27: value 100 n -> 2.2u, 63V; device passives:C0603 -> passives:E2,0-6
- C30: value 10u, 16V -> 2.2u, 63V; device passives:SV-A -> passives:E2,0-6
- C31: value 10u, 16V -> 390 u / 63 V; device passives:SV-A -> passives:E5,0-12,5
- C33, CH1:C6, CH1:C7, CH2:C6, CH2:C7, CH3:C6, CH3:C7: value 33u, 63V -> 10u; device passives:SV-E/F -> passives:E2,0-5
- CH1:C1, CH1:C2, CH2:C1, CH2:C2, CH3:C1, CH3:C2: value (none) -> 10u, 63V; device passives:C0603 -> passives:E2,0-6
- CH1:C3, CH1:C5, CH2:C3, CH2:C5, CH3:C3, CH3:C5: value (none) -> 10u; device passives:C0603 -> passives:E2,0-5
- CH1:GAIN1, CH1:GAIN2, CH2:GAIN1, CH2:GAIN2, CH3:GAIN1, CH3:GAIN2, GAIN1, GAIN2, GAIN3, GAIN4: device passives:ECP10P -> passives:RJ9W
- CH1:R10, CH1:R11, CH1:R12, CH1:R13, CH1:R14, CH1:R15, CH1:R16, CH1:R17, CH1:R18, CH1:R19, CH1:R20, CH1:R21, CH1:R22, CH1:R23, CH1:R24, CH1:R25, CH1:R26, CH1:R27, CH1:R8, CH1:R9, CH2:R10, CH2:R11, CH2:R12, CH2:R13, CH2:R14, CH2:R15, CH2:R16, CH2:R17, CH2:R18, CH2:R19, CH2:R20, CH2:R21, CH2:R22, CH2:R23, CH2:R24, CH2:R25, CH2:R26, CH2:R27, CH2:R8, CH2:R9, CH3:R10, CH3:R11, CH3:R12, CH3:R13, CH3:R14, CH3:R15, CH3:R16, CH3:R17, CH3:R18, CH3:R19, CH3:R20, CH3:R21, CH3:R22, CH3:R23, CH3:R24, CH3:R25, CH3:R26, CH3:R27, CH3:R8, CH3:R9, R1, R10, R11, R12, R13, R14, R15, R16, R17, R18, R19, R2, R20, R21, R22, R23, R24, R25, R26, R27, R28, R29, R3, R30, R31, R32, R33, R34, R35, R36, R37, R38, R39, R4, R40, R41, R42, R43, R44, R45, R46, R47, R48, R49, R5, R50, R51, R52, R53, R54, R55, R56, R57, R58, R59, R6, R60, R61, R62, R63, R7, R8, R9: device passives:R0603 -> passives:0204/7
- CH1:U1, CH2:U1, CH3:U1, U1, U2, U3, U4, U5, U6, U7: value TL074IDT -> TL074; device ic:SOIC127P600X175-14N -> ic:DIP762W53P254L1969H508Q14B
- CH1:U2, CH2:U2, CH3:U2: value TL074IDT -> SEND_RETURN; device ic:SOIC127P600X175-14N -> connectors:SND_RET
- U$1: value UTBULT_DESIGN4 -> UTBULT_DESIGN3; device misc:UD_4 -> misc:UD_3
- moved R20 1177.3 mm to (-141.6, 181.4), flipped to the bottom
- moved R19 1171.4 mm to (-151.7, 181.4), flipped to the bottom
- moved PWR$1 1166.4 mm to (5.69, 112.1), flipped to the bottom
- moved C4 1159.5 mm to (-47.6, 164.8), flipped to the bottom
- moved VOLUM6 1150.1 mm to (119.0, 48.0)
- moved C3 1147.8 mm to (-57.8, 164.8), flipped to the bottom
- moved U7 1140.1 mm to (-121.3, 109.0), flipped to the bottom
- moved R17 1139.8 mm to (-172.1, 181.4), flipped to the bottom
- moved R16 1134.0 mm to (-182.2, 181.4), flipped to the bottom
- moved U6 1132.4 mm to (-131.4, 109.0), flipped to the bottom
- moved U5 1128.8 mm to (-141.6, 109.0), flipped to the bottom
- moved C2 1121.4 mm to (-67.9, 164.8), flipped to the bottom
- moved C1 1109.9 mm to (-78.1, 164.8), flipped to the bottom
- moved R24 1103.9 mm to (-100.9, 181.4), flipped to the bottom
- moved R23 1103.9 mm to (-111.1, 181.4), flipped to the bottom
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Connections:
- removed net CH1:EQ_IN: CH1:C12.-, CH1:R5.1, CH1:U2.3
- removed net CH1:N$10: CH1:FRQ1.P$3, CH1:R3.2
- removed net CH1:N$13: CH1:C12.+, CH1:R22.1, CH1:U1.14
- removed net CH1:N$16: CH1:C3.1, CH1:FR2.P$2
- removed net CH1:N$18: CH1:C5.2, CH1:Q2.P$1, CH1:Q2.P$2, CH1:R4.2
- removed net CH1:N$19: CH1:C3.2, CH1:Q2.P$3
- removed net CH1:N$20: CH1:R4.1, CH1:U2.8, CH1:U2.9
- removed net CH1:N$21: CH1:C5.1, CH1:R6.1, CH1:U2.10
- removed net CH1:N$22: CH1:FRQ2.P$3, CH1:R6.2
- removed net CH1:N$3: CH1:C1.2, CH1:FR1.P$2
- removed net CH1:N$32: CH1:C18.+, CH1:R13.2
- removed net CH1:N$35: CH1:C20.+, CH1:R15.2
- removed net CH1:N$4: CH1:FR1.P$3, CH1:FR2.P$3, CH1:R7.2, CH1:U2.13
- removed net CH1:N$5: CH1:C1.1, CH1:Q1.P$3
- removed net CH1:N$6: CH1:C2.2, CH1:Q1.P$1, CH1:Q1.P$2, CH1:R2.2
- removed net CH1:N$7: CH1:R2.1, CH1:U2.6, CH1:U2.7
- removed net CH1:N$8: CH1:C2.1, CH1:R3.1, CH1:U2.5
- removed net CH2:EQ_IN: CH2:C12.-, CH2:R5.1, CH2:U2.3
- removed net CH2:N$10: CH2:FRQ1.P$3, CH2:R3.2
- removed net CH2:N$13: CH2:C12.+, CH2:R22.1, CH2:U1.14
- removed net CH2:N$16: CH2:C3.1, CH2:FR2.P$2
- removed net CH2:N$18: CH2:C5.2, CH2:Q2.P$1, CH2:Q2.P$2, CH2:R4.2
- removed net CH2:N$19: CH2:C3.2, CH2:Q2.P$3
- removed net CH2:N$20: CH2:R4.1, CH2:U2.8, CH2:U2.9
- removed net CH2:N$21: CH2:C5.1, CH2:R6.1, CH2:U2.10
- removed net CH2:N$22: CH2:FRQ2.P$3, CH2:R6.2
- removed net CH2:N$3: CH2:C1.2, CH2:FR1.P$2
- removed net CH2:N$32: CH2:C18.+, CH2:R13.2
- removed net CH2:N$35: CH2:C20.+, CH2:R15.2
- removed net CH2:N$4: CH2:FR1.P$3, CH2:FR2.P$3, CH2:R7.2, CH2:U2.13
- removed net CH2:N$5: CH2:C1.1, CH2:Q1.P$3
- removed net CH2:N$6: CH2:C2.2, CH2:Q1.P$1, CH2:Q1.P$2, CH2:R2.2
- removed net CH2:N$7: CH2:R2.1, CH2:U2.6, CH2:U2.7
- removed net CH2:N$8: CH2:C2.1, CH2:R3.1, CH2:U2.5
- removed net CH3:EQ_IN: CH3:C12.-, CH3:R5.1, CH3:U2.3
- removed net CH3:N$10: CH3:FRQ1.P$3, CH3:R3.2
- removed net CH3:N$13: CH3:C12.+, CH3:R22.1, CH3:U1.14
- removed net CH3:N$16: CH3:C3.1, CH3:FR2.P$2
- removed net CH3:N$18: CH3:C5.2, CH3:Q2.P$1, CH3:Q2.P$2, CH3:R4.2
- removed net CH3:N$19: CH3:C3.2, CH3:Q2.P$3
- removed net CH3:N$20: CH3:R4.1, CH3:U2.8, CH3:U2.9
- removed net CH3:N$21: CH3:C5.1, CH3:R6.1, CH3:U2.10
- removed net CH3:N$22: CH3:FRQ2.P$3, CH3:R6.2
- removed net CH3:N$3: CH3:C1.2, CH3:FR1.P$2
- removed net CH3:N$32: CH3:C18.+, CH3:R13.2
- removed net CH3:N$35: CH3:C20.+, CH3:R15.2
- removed net CH3:N$4: CH3:FR1.P$3, CH3:FR2.P$3, CH3:R7.2, CH3:U2.13
- removed net CH3:N$5: CH3:C1.1, CH3:Q1.P$3
- removed net CH3:N$6: CH3:C2.2, CH3:Q1.P$1, CH3:Q1.P$2, CH3:R2.2
- removed net CH3:N$7: CH3:R2.1, CH3:U2.6, CH3:U2.7
- removed net CH3:N$8: CH3:C2.1, CH3:R3.1, CH3:U2.5
- removed net RET_L: VOLUME1.P$3
- removed net RET_R: VOLUME1.P$8
- removed net SEL_DRY: C13.+, R18.2
- removed net TC_DRY: BLEND1.P$2, BLEND1.P$7, R3.2, R6.2
- new net MASTER_MON_L: U$6.D2, VOLUM6.P$3, VOLUME1.P$8
- new net MASTER_MON_R: U$6.D1, VOLUM6.P$8, VOLUME1.P$3
- new net N$65: U$6.S1B, U8.1, U8.2
- new net N$70: D1.A, U9.3
- new net N$71: U$6.S2B, U8.6, U8.7
- new net N$72: MONO.P$3, VOLUM6.P$7
- new net N$73: C28.1, R45.2, R46.1, U7.12
- new net N$74: LD1.CR, U$5.S4B
- new net N$75: LD1.CX, U$5.S4A
- new net N$76: R64.1, U$5.D4
- new net N$79: C27.+, U$10.P$1, U9.1
- new net N$81: D2.A, PWR$1.P$1
- new net SELECT: BYPASS.P$2, R65.2, U$5.IN1, U$5.IN2, U$5.IN3, U$5.IN4, U$6.IN1, U$6.IN2
- new net TC_BALANCED: BLEND1.P$2, BLEND1.P$7, R3.2, R6.2, U8.10, U8.12
- new net TC_BYPASS_L: TC_RET.BPSR, U8.8, U8.9
- new net TC_BYPASS_R: TC_RET.BPSL, U8.13, U8.14
- net +48V: now also C30.+, C31.+, U$10.P$2
- net +9V: now also BYPASS.P$1, D1.C, D2.C, R64.2, U$5.VDD, U$6.VDD, U8.4; no longer C11.1, C26.1, C27.1, C37.1, C40.1, C41.1, C42.1, CH1:C10.2, CH1:U2.4, CH2:C10.2, CH2:U2.4, CH3:C10.2, CH3:U2.4, PWR$1.P$1
- net CH1:COLD_IN: now also CH1:C1.+, CH1:IN.P$3; no longer CH1:C7.+, CH1:TC.P$3
- net CH1:COLD_SEND: now also CH1:C3.+; no longer CH1:C8.+
- net CH1:HOT_IN: now also CH1:C2.+, CH1:IN.P$2; no longer CH1:C6.+, CH1:TC.P$2
- net CH1:HOT_SEND: now also CH1:C5.+; no longer CH1:C9.+
- net CH1:N$1: now also CH1:C10.+, CH1:R13.2; no longer CH1:R1.2, CH1:U2.1, CH1:U2.2
- net CH1:N$14: now also CH1:C1.-, CH1:C3.-; no longer CH1:C7.-, CH1:C8.-
- net CH1:N$15: now also CH1:C2.-, CH1:C5.-; no longer CH1:C6.-, CH1:C9.-
- net CH1:N$2: now also CH1:C12.+, CH1:R15.2; no longer CH1:FR1.P$1, CH1:FR2.P$1, CH1:R1.1, CH1:U2.12
- net CH1:N$23: now also CH1:C6.-, CH1:C7.-; no longer CH1:C13.-, CH1:C14.-
- net CH1:N$24: no longer CH1:C10.1, CH1:U2.11
- net CH1:N$25: now also CH1:C6.+, CH1:U2.P$1; no longer CH1:C14.+, CH1:U$1.P$1
- net CH1:N$26: now also CH1:C8.-, CH1:C9.-; no longer CH1:C15.-, CH1:C16.-
- net CH1:N$27: now also CH1:C8.+, CH1:U2.P$2; no longer CH1:C15.+, CH1:U$1.P$2
- net CH1:N$28: now also CH1:C9.+; no longer CH1:C16.+
- net CH1:N$37: now also CH1:BLEND.P$8; no longer CH1:BLEND1.P$8
- net CH1:SND_RET_OUT: now also CH1:BLEND.P$1; no longer CH1:BLEND1.P$1
- net CH2:COLD_IN: now also CH2:C1.+, CH2:IN.P$3; no longer CH2:C7.+, CH2:TC.P$3
- net CH2:COLD_SEND: now also CH2:C3.+; no longer CH2:C8.+
- net CH2:HOT_IN: now also CH2:C2.+, CH2:IN.P$2; no longer CH2:C6.+, CH2:TC.P$2
- net CH2:HOT_SEND: now also CH2:C5.+; no longer CH2:C9.+
- net CH2:N$1: now also CH2:C10.+, CH2:R13.2; no longer CH2:R1.2, CH2:U2.1, CH2:U2.2
- net CH2:N$14: now also CH2:C1.-, CH2:C3.-; no longer CH2:C7.-, CH2:C8.-
- net CH2:N$15: now also CH2:C2.-, CH2:C5.-; no longer CH2:C6.-, CH2:C9.-
- net CH2:N$2: now also CH2:C12.+, CH2:R15.2; no longer CH2:FR1.P$1, CH2:FR2.P$1, CH2:R1.1, CH2:U2.12
- net CH2:N$23: now also CH2:C6.-, CH2:C7.-; no longer CH2:C13.-, CH2:C14.-
- net CH2:N$24: no longer CH2:C10.1, CH2:U2.11
- net CH2:N$25: now also CH2:C6.+, CH2:U2.P$1; no longer CH2:C14.+, CH2:U$1.P$1
- net CH2:N$26: now also CH2:C8.-, CH2:C9.-; no longer CH2:C15.-, CH2:C16.-
- net CH2:N$27: now also CH2:C8.+, CH2:U2.P$2; no longer CH2:C15.+, CH2:U$1.P$2
- net CH2:N$28: now also CH2:C9.+; no longer CH2:C16.+
- net CH2:N$37: now also CH2:BLEND.P$8; no longer CH2:BLEND1.P$8
- net CH2:SND_RET_OUT: now also CH2:BLEND.P$1; no longer CH2:BLEND1.P$1
- net CH3:COLD_IN: now also CH3:C1.+, CH3:IN.P$3; no longer CH3:C7.+, CH3:TC.P$3
- net CH3:COLD_SEND: now also CH3:C3.+; no longer CH3:C8.+
- net CH3:HOT_IN: now also CH3:C2.+, CH3:IN.P$2; no longer CH3:C6.+, CH3:TC.P$2
- net CH3:HOT_SEND: now also CH3:C5.+; no longer CH3:C9.+
- net CH3:N$1: now also CH3:C10.+, CH3:R13.2; no longer CH3:R1.2, CH3:U2.1, CH3:U2.2
- net CH3:N$14: now also CH3:C1.-, CH3:C3.-; no longer CH3:C7.-, CH3:C8.-
- net CH3:N$15: now also CH3:C2.-, CH3:C5.-; no longer CH3:C6.-, CH3:C9.-
- net CH3:N$2: now also CH3:C12.+, CH3:R15.2; no longer CH3:FR1.P$1, CH3:FR2.P$1, CH3:R1.1, CH3:U2.12
- net CH3:N$23: now also CH3:C6.-, CH3:C7.-; no longer CH3:C13.-, CH3:C14.-
- net CH3:N$24: no longer CH3:C10.1, CH3:U2.11
- net CH3:N$25: now also CH3:C6.+, CH3:U2.P$1; no longer CH3:C14.+, CH3:U$1.P$1
- net CH3:N$26: now also CH3:C8.-, CH3:C9.-; no longer CH3:C15.-, CH3:C16.-
- net CH3:N$27: now also CH3:C8.+, CH3:U2.P$2; no longer CH3:C15.+, CH3:U$1.P$2
- net CH3:N$28: now also CH3:C9.+; no longer CH3:C16.+
- net CH3:N$37: now also CH3:BLEND.P$8; no longer CH3:BLEND1.P$8
- net CH3:SND_RET_OUT: now also CH3:BLEND.P$1; no longer CH3:BLEND1.P$1
- net COLD_SEND: now also C11.+; no longer C30.+
- net DRY1: now also CH1:C7.+, CH1:R22.1, CH1:U1.14, U$5.S1B; no longer CH1:C13.+, CH1:R7.1, CH1:U2.14
- net DRY2: now also CH2:C7.+, CH2:R22.1, CH2:U1.14, U$5.S2B; no longer CH2:C13.+, CH2:R7.1, CH2:U2.14
- net DRY3: now also CH3:C7.+, CH3:R22.1, CH3:U1.14, U$5.S3B; no longer CH3:C13.+, CH3:R7.1, CH3:U2.14
- net GND: now also BYPASS.P$3, C27.-, C30.-, C31.-, C33.-, CH1:BLEND.P$4, CH1:BLEND.P$5, CH1:C10.-, CH1:C12.-, CH1:IN.P$1, CH1:LEVEL.P$4, CH1:LEVEL.P$5, CH1:U2.P$3, CH2:BLEND.P$4, CH2:BLEND.P$5, CH2:C10.-, CH2:C12.-, CH2:IN.P$1, CH2:LEVEL.P$4, CH2:LEVEL.P$5, CH2:U2.P$3, CH3:BLEND.P$4, CH3:BLEND.P$5, CH3:C10.-, CH3:C12.-, CH3:IN.P$1, CH3:LEVEL.P$4, CH3:LEVEL.P$5, CH3:U2.P$3, LD1.A, LOOPMASTER.P$3, MON_IN.P$1, MON_OUT.P$1, MON_THROUGH.P$1, OUT_L.P$1, OUT_R.P$1, R65.1, TC_RET.GND, TC_SEND_JACK.P$1, U$5.GND, U$5.VSS, U$6.GND, U$6.VSS, U8.11, U9.2; no longer C11.2, C26.2, C27.2, C39.-, C40.2, C41.2, C42.2, CH1:BLEND1.P$4, CH1:BLEND1.P$5, CH1:C18.-, CH1:C20.-, CH1:FR1.P$4, CH1:FR1.P$5, CH1:FR2.P$4, CH1:FR2.P$5, CH1:FRQ1.P$4, CH1:FRQ1.P$5, CH1:FRQ2.P$4, CH1:FRQ2.P$5, CH1:Q1.P$4, CH1:Q1.P$5, CH1:Q2.P$4, CH1:Q2.P$5, CH1:R5.2, CH1:TC.P$1, CH1:U$1.P$3, CH1:U$2.P$4, CH1:U$2.P$5, CH2:BLEND1.P$4, CH2:BLEND1.P$5, CH2:C18.-, CH2:C20.-, CH2:FR1.P$4, CH2:FR1.P$5, CH2:FR2.P$4, CH2:FR2.P$5, CH2:FRQ1.P$4, CH2:FRQ1.P$5, CH2:FRQ2.P$4, CH2:FRQ2.P$5, CH2:Q1.P$4, CH2:Q1.P$5, CH2:Q2.P$4, CH2:Q2.P$5, CH2:R5.2, CH2:TC.P$1, CH2:U$1.P$3, CH2:U$2.P$4, CH2:U$2.P$5, CH3:BLEND1.P$4, CH3:BLEND1.P$5, CH3:C18.-, CH3:C20.-, CH3:FR1.P$4, CH3:FR1.P$5, CH3:FR2.P$4, CH3:FR2.P$5, CH3:FRQ1.P$4, CH3:FRQ1.P$5, CH3:FRQ2.P$4, CH3:FRQ2.P$5, CH3:Q1.P$4, CH3:Q1.P$5, CH3:Q2.P$4, CH3:Q2.P$5, CH3:R5.2, CH3:TC.P$1, CH3:U$1.P$3, CH3:U$2.P$4, CH3:U$2.P$5, GAIN.P$4, GAIN.P$5, TC.P$1, TC1.P$1, TC2.P$1, TC3.P$1, U$2.P$3, U$3.P$1, U$4.P$1
- net HOT_SEND: now also C26.+; no longer C31.+
- net L_COLD: now also OUT_L.P$3; no longer TC1.P$3
- net L_HOT: now also OUT_L.P$2; no longer TC1.P$2
- net MIX1: now also CH1:LEVEL.P$2; no longer CH1:U$2.P$2
- net MIX2: now also CH2:LEVEL.P$2; no longer CH2:U$2.P$2
- net MIX3: now also CH3:LEVEL.P$2; no longer CH3:U$2.P$2
- net MIX_OUT: now also R18.2, U8.3, U8.5
- net MON_COLD: now also C25.+, MON_IN.P$3, MON_THROUGH.P$3; no longer C33.+, TC3.P$3
- net MON_HOT: now also MON_IN.P$2, MON_THROUGH.P$2; no longer TC3.P$2
- net MON_OUT_L: now also MON_OUT.P$2; no longer U$4.P$2
- net MON_OUT_R: now also MON_OUT.P$3; no longer U$4.P$3
- net N$12: now also C2.-; no longer C3.-
- net N$14: now also C6.-; no longer C7.-
- net N$15: now also C7.-; no longer C6.-
- net N$23: no longer C13.-
- net N$25: now also C11.-, C25.-; no longer C30.-, C33.-
- net N$27: now also C26.-; no longer C31.-
- net N$42: now also C13.-, C23.-; no longer C22.-, C25.-
- net N$43: now also C22.-; no longer C23.-
- net N$44: now also C13.+; no longer C22.+
- net N$45: now also C22.+; no longer C23.+
- net N$46: now also GAIN5.E; no longer GAIN.P$3
- net N$50: now also GAIN5.S; no longer GAIN.P$2
- net N$51: now also MONO.P$1
- net N$58: now also MONO.P$2; no longer VOLUM6.P$7
- net N$63: now also C33.+; no longer C36.+
- net N$68: now also C36.+; no longer C39.+
- net N$9: now also C3.-; no longer C2.-
- net OUT_L: now also VOLUME1.P$7; no longer VOLUME1.P$2
- net OUT_R: now also VOLUME1.P$2; no longer VOLUME1.P$7
- net RET: now also LOOPMASTER.P$2; no longer U$2.P$2
- net RET1: now also CH1:LEVEL.P$3, U$5.D1; no longer CH1:U$2.P$3
- net RET2: now also CH2:LEVEL.P$3, U$5.D2; no longer CH2:U$2.P$3
- net RET3: now also CH3:LEVEL.P$3, U$5.D3; no longer CH3:U$2.P$3
- net R_COLD: now also OUT_R.P$3; no longer TC2.P$3
- net R_HOT: now also C23.+, OUT_R.P$2; no longer C25.+, TC2.P$2
- net SND: now also LOOPMASTER.P$1; no longer U$2.P$1
- net TC_COLD: now also C7.+, TC_SEND_JACK.P$3; no longer C6.+, TC.P$3
- net TC_HOT: now also C6.+, TC_SEND_JACK.P$2; no longer C7.+, TC.P$2
- net TC_RET_L: now also TC_RET.LEFT; no longer U$3.P$2
- net TC_RET_R: now also C2.+, TC_RET.RIGHT; no longer C3.+, U$3.P$3
- net TC_WET_L: now also C3.+, U$6.S1A; no longer C2.+, VOLUM6.P$3
- net TC_WET_R: now also U$6.S2A; no longer VOLUM6.P$8
- net VDD: now also C37.1, CH1:BLEND.P$3, CH1:BLEND.P$6, CH1:LEVEL.P$1, CH2:BLEND.P$3, CH2:BLEND.P$6, CH2:LEVEL.P$1, CH3:BLEND.P$3, CH3:BLEND.P$6, CH3:LEVEL.P$1, U7.13, U7.14; no longer C28.1, CH1:BLEND1.P$3, CH1:BLEND1.P$6, CH1:FRQ1.P$1, CH1:FRQ1.P$2, CH1:FRQ2.P$1, CH1:FRQ2.P$2, CH1:U$2.P$1, CH2:BLEND1.P$3, CH2:BLEND1.P$6, CH2:FRQ1.P$1, CH2:FRQ1.P$2, CH2:FRQ2.P$1, CH2:FRQ2.P$2, CH2:U$2.P$1, CH3:BLEND1.P$3, CH3:BLEND1.P$6, CH3:FRQ1.P$1, CH3:FRQ1.P$2, CH3:FRQ2.P$1, CH3:FRQ2.P$2, CH3:U$2.P$1, R45.2, R46.1
- net WET1: now also CH1:BLEND.P$2, CH1:BLEND.P$7, U$5.S1A; no longer CH1:BLEND1.P$2, CH1:BLEND1.P$7
- net WET2: now also CH2:BLEND.P$2, CH2:BLEND.P$7, U$5.S2A; no longer CH2:BLEND1.P$2, CH2:BLEND1.P$7
- net WET3: now also CH3:BLEND.P$2, CH3:BLEND.P$7, U$5.S3A; no longer CH3:BLEND1.P$2, CH3:BLEND1.P$7
Routing:
- net +48V: track 0.00 -> 55.9 mm, vias 0 -> 2
Other:
- board size 190 x 190 mm -> 142 x 128 mm
- board text added: "Blend"
- board text added: "Bypass"
- board text added: "Chanel 1"
- board text added: "Chanel 2"
- board text added: "Chanel 3"
- board text added: "D"
- board text added: "Dry"
- board text added: "Gain"
- board text added: "Input 1"
- board text added: "Input 2"
- board text added: "Input 3"
- board text added: "L"
- board text added: "Left Out"
- board text added: "Level"
- board text added: "Loop 1"
- board text added: "Loop 2"
- board text added: "Loop 3"
- board text added: "Loop master"
- board text added: "M"
- board text added: "Master"
- board text added: "Mon in gain"
- board text added: "Mon out gain"
- board text added: "Monitor"
- board text added: "Monitor Through"
- board text added: "Monitor in"
- board text added: "Monitor out"
- board text added: "Mono"
- board text added: "Power"
- board text added: "R"
- board text added: "Right Out"
- board text added: "S"
- board text added: "TC return"
- board text added: "TC send"
- board text added: "W"
- board text added: "Wet"
- board text added: "ret"

Commit message: Added internal bondary
Parts:
- moved CH3:C3 262.2 mm to (113.0, 84.3), turned to 90 degrees
- moved CH3:C5 255.6 mm to (119.1, 81.9), turned to 90 degrees
- moved CH3:U1 255.0 mm to (72.3, 82.5)
- moved CH2:U1 246.8 mm to (55.9, 88.8), turned to 90 degrees
- moved CH1:C3 246.7 mm to (81.0, 85.7), turned to 90 degrees
- moved CH2:C3 245.1 mm to (91.2, 88.2), turned to 90 degrees
- moved CH1:U1 243.9 mm to (39.4, 82.6)
- moved CH3:R16 241.0 mm to (109.2, 76.2), turned to 180 degrees
- moved CH1:C5 239.6 mm to (83.6, 92.0), turned to 90 degrees
- moved CH3:R26 239.5 mm to (66.1, 100.3), turned to 180 degrees
- moved CH2:C5 238.9 mm to (97.5, 88.2), turned to 90 degrees
- moved CH2:R16 233.7 mm to (99.7, 79.8)
- moved CH3:R17 231.0 mm to (109.2, 73.6), turned to 180 degrees
- moved CH1:R16 230.8 mm to (86.3, 78.7), turned to 90 degrees
- moved CH2:R17 224.0 mm to (99.7, 82.3)
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Routing:
- net +48V: track 55.9 -> 0.00 mm, vias 2 -> 0

Commit message: Swapped gain trimpots and started restructuring
Parts:
- removed CH1:C1, CH1:C2, CH2:C1, CH2:C2, CH3:C1, CH3:C2: 10u, 63V, passives:E2,0-6
- removed CH1:C10, CH1:C12, CH1:C3, CH1:C5, CH1:C6, CH1:C7, CH1:C8, CH1:C9, CH2:C10, CH2:C12, CH2:C3, CH2:C5, CH2:C6, CH2:C7, CH2:C8, CH2:C9, CH3:C10, CH3:C12, CH3:C3, CH3:C5, CH3:C6, CH3:C7, CH3:C8, CH3:C9: 10u, passives:E2,0-5
- removed CH1:C11, CH2:C11, CH3:C11: 100 n, passives:C025-025X050
- removed CH1:C17, CH1:C19, CH1:C4, CH2:C17, CH2:C19, CH2:C4, CH3:C17, CH3:C19, CH3:C4: 18 p, passives:C025-025X050
- removed CH1:R10, CH1:R16, CH1:R17, CH1:R23, CH1:R24, CH1:R8, CH1:R9, CH2:R10, CH2:R16, CH2:R17, CH2:R23, CH2:R24, CH2:R8, CH2:R9, CH3:R10, CH3:R16, CH3:R17, CH3:R23, CH3:R24, CH3:R8, CH3:R9: 100 k, passives:0204/7
- removed CH1:R11, CH1:R14, CH2:R11, CH2:R14, CH3:R11, CH3:R14: 47 k, passives:0204/7
- removed CH1:R12, CH1:R18, CH1:R26, CH2:R12, CH2:R18, CH2:R26, CH3:R12, CH3:R18, CH3:R26: 1 k, passives:0204/7
- removed CH1:R13, CH1:R15, CH2:R13, CH2:R15, CH3:R13, CH3:R15: 2.2 k, passives:0204/7
- removed CH1:R19, CH1:R20, CH1:R21, CH1:R22, CH2:R19, CH2:R20, CH2:R21, CH2:R22, CH3:R19, CH3:R20, CH3:R21, CH3:R22: 10 k, passives:0204/7
- removed CH1:R25, CH1:R27, CH2:R25, CH2:R27, CH3:R25, CH3:R27: 4.7 k, passives:0204/7
- removed CH1:U1, CH2:U1, CH3:U1: TL074, ic:DIP762W53P254L1969H508Q14B
- added 1:C1, 1:C2, 2:C1, 2:C2, 3:C1, 3:C2: 10u, 63V, passives:E2,0-6
- added 1:C10, 1:C12, 1:C3, 1:C5, 1:C6, 1:C7, 1:C8, 1:C9, 2:C10, 2:C12, 2:C3, 2:C5, 2:C6, 2:C7, 2:C8, 2:C9, 3:C10, 3:C12, 3:C3, 3:C5, 3:C6, 3:C7, 3:C8, 3:C9: 10u, passives:E2,0-5
- added 1:C11, 2:C11, 3:C11: 100 n, passives:C025-025X050
- added 1:C17, 1:C19, 1:C4, 2:C17, 2:C19, 2:C4, 3:C17, 3:C19, 3:C4: 18 p, passives:C025-025X050
- added 1:R10, 1:R16, 1:R17, 1:R23, 1:R24, 1:R8, 1:R9, 2:R10, 2:R16, 2:R17, 2:R23, 2:R24, 2:R8, 2:R9, 3:R10, 3:R16, 3:R17, 3:R23, 3:R24, 3:R8, 3:R9: 100 k, passives:0204/7
- added 1:R11, 1:R14, 2:R11, 2:R14, 3:R11, 3:R14: 47 k, passives:0204/7
- added 1:R12, 1:R18, 1:R26, 2:R12, 2:R18, 2:R26, 3:R12, 3:R18, 3:R26: 1 k, passives:0204/7
- added 1:R13, 1:R15, 2:R13, 2:R15, 3:R13, 3:R15: 2.2 k, passives:0204/7
- added 1:R19, 1:R20, 1:R21, 1:R22, 2:R19, 2:R20, 2:R21, 2:R22, 3:R19, 3:R20, 3:R21, 3:R22: 10 k, passives:0204/7
- added 1:R25, 1:R27, 2:R25, 2:R27, 3:R25, 3:R27: 4.7 k, passives:0204/7
- added 1:U1, 2:U1, 3:U1: TL074, ic:DIP762W53P254L1969H508Q14B
- added U$2: UNBALANCED_INPUT_JACK, connectors:BALANCED_INPUT_JACK
- moved R30 80.8 mm to (-205.1, 263.9)
- moved R35 80.8 mm to (-154.3, 263.9)
- moved R36 80.8 mm to (-144.1, 263.9)
- moved R37 80.8 mm to (-134.0, 263.9)
- moved R38 80.8 mm to (-123.8, 263.9)
- moved R39 80.8 mm to (-113.6, 263.9)
- moved R40 80.8 mm to (-103.5, 263.9)
- moved R41 80.8 mm to (-93.3, 263.9)
- moved R42 80.8 mm to (-83.2, 263.9)
- moved R43 80.8 mm to (-73.0, 263.9)
- moved R31 80.8 mm to (-194.9, 263.9)
- moved R32 80.8 mm to (-184.8, 263.9)
- moved R33 80.8 mm to (-174.6, 263.9)
- moved R34 80.8 mm to (-164.4, 263.9)
- moved U$5 80.8 mm to (-205.1, 187.7)
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- renumbered CH1:BLEND to 1:BLEND, CH1:GAIN to 1:GAIN, CH1:GAIN1 to 1:GAIN1, CH1:GAIN2 to 1:GAIN2, CH1:IN to 1:IN, CH1:LEVEL to 1:LEVEL, CH1:U2 to 1:U2, CH2:BLEND to 2:BLEND, CH2:GAIN to 2:GAIN, CH2:GAIN1 to 2:GAIN1, CH2:GAIN2 to 2:GAIN2, CH2:IN to 2:IN, CH2:LEVEL to 2:LEVEL, CH2:U2 to 2:U2, CH3:BLEND to 3:BLEND, CH3:GAIN to 3:GAIN, CH3:GAIN1 to 3:GAIN1, CH3:GAIN2 to 3:GAIN2, CH3:IN to 3:IN, CH3:LEVEL to 3:LEVEL, CH3:U2 to 3:U2
Connections:
- removed net CH1:COLD_IN: 1:IN.P$3, CH1:C1.+, CH1:R27.2
- removed net CH1:COLD_SEND: CH1:C3.+, CH1:R16.2, CH1:U1.10
- removed net CH1:HOT_IN: 1:IN.P$2, CH1:C2.+, CH1:R25.2
- removed net CH1:HOT_SEND: CH1:C5.+, CH1:R17.2, CH1:U1.12
- removed net CH1:N$1: CH1:C10.+, CH1:R13.2
- removed net CH1:N$11: CH1:C4.1, CH1:R19.1
- removed net CH1:N$12: CH1:C4.2, CH1:R20.1, CH1:R22.2, CH1:R26.1, CH1:U1.13
- removed net CH1:N$14: CH1:C1.-, CH1:C3.-, CH1:R23.2
- removed net CH1:N$15: CH1:C2.-, CH1:C5.-, CH1:R24.2
- removed net CH1:N$17: 1:GAIN.P$2, CH1:R26.2
- removed net CH1:N$2: CH1:C12.+, CH1:R15.2
- removed net CH1:N$23: CH1:C6.-, CH1:C7.-, CH1:R8.2
- removed net CH1:N$24: CH1:C11.1, CH1:U1.11
- removed net CH1:N$25: 1:U2.P$1, CH1:C6.+
- removed net CH1:N$26: CH1:C8.-, CH1:C9.-, CH1:R9.2
- removed net CH1:N$27: 1:U2.P$2, CH1:C8.+
- removed net CH1:N$28: CH1:C9.+, CH1:R10.2, CH1:R12.2
- removed net CH1:N$29: 1:GAIN1.A, CH1:C17.2, CH1:R11.2, CH1:U1.2
- removed net CH1:N$30: 1:GAIN2.A, CH1:C19.2, CH1:R14.2, CH1:U1.6
- removed net CH1:N$31: 1:GAIN1.E, 1:GAIN1.S, CH1:R13.1
- removed net CH1:N$33: CH1:R12.1, CH1:U1.3
- removed net CH1:N$34: 1:GAIN2.E, 1:GAIN2.S, CH1:R15.1
- removed net CH1:N$36: CH1:R18.1, CH1:U1.5
- removed net CH1:N$37: 1:BLEND.P$8, CH1:C19.1, CH1:R14.1, CH1:U1.7
- removed net CH1:N$9: 1:GAIN.P$3, CH1:R19.2, CH1:R20.2, CH1:R21.1, CH1:U1.8, CH1:U1.9
- removed net CH1:SND_RET_OUT: 1:BLEND.P$1, CH1:C17.1, CH1:R11.1, CH1:U1.1
- removed net CH2:COLD_IN: 2:IN.P$3, CH2:C1.+, CH2:R27.2
- removed net CH2:COLD_SEND: CH2:C3.+, CH2:R16.2, CH2:U1.10
- removed net CH2:HOT_IN: 2:IN.P$2, CH2:C2.+, CH2:R25.2
- removed net CH2:HOT_SEND: CH2:C5.+, CH2:R17.2, CH2:U1.12
- removed net CH2:N$1: CH2:C10.+, CH2:R13.2
- removed net CH2:N$11: CH2:C4.1, CH2:R19.1
- removed net CH2:N$12: CH2:C4.2, CH2:R20.1, CH2:R22.2, CH2:R26.1, CH2:U1.13
- removed net CH2:N$14: CH2:C1.-, CH2:C3.-, CH2:R23.2
- removed net CH2:N$15: CH2:C2.-, CH2:C5.-, CH2:R24.2
- removed net CH2:N$17: 2:GAIN.P$2, CH2:R26.2
- removed net CH2:N$2: CH2:C12.+, CH2:R15.2
- removed net CH2:N$23: CH2:C6.-, CH2:C7.-, CH2:R8.2
- removed net CH2:N$24: CH2:C11.1, CH2:U1.11
- removed net CH2:N$25: 2:U2.P$1, CH2:C6.+
- removed net CH2:N$26: CH2:C8.-, CH2:C9.-, CH2:R9.2
- removed net CH2:N$27: 2:U2.P$2, CH2:C8.+
- removed net CH2:N$28: CH2:C9.+, CH2:R10.2, CH2:R12.2
- removed net CH2:N$29: 2:GAIN1.A, CH2:C17.2, CH2:R11.2, CH2:U1.2
- removed net CH2:N$30: 2:GAIN2.A, CH2:C19.2, CH2:R14.2, CH2:U1.6
- removed net CH2:N$31: 2:GAIN1.E, 2:GAIN1.S, CH2:R13.1
- removed net CH2:N$33: CH2:R12.1, CH2:U1.3
- removed net CH2:N$34: 2:GAIN2.E, 2:GAIN2.S, CH2:R15.1
- removed net CH2:N$36: CH2:R18.1, CH2:U1.5
- removed net CH2:N$37: 2:BLEND.P$8, CH2:C19.1, CH2:R14.1, CH2:U1.7
- removed net CH2:N$9: 2:GAIN.P$3, CH2:R19.2, CH2:R20.2, CH2:R21.1, CH2:U1.8, CH2:U1.9
- removed net CH2:SND_RET_OUT: 2:BLEND.P$1, CH2:C17.1, CH2:R11.1, CH2:U1.1
- removed net CH3:COLD_IN: 3:IN.P$3, CH3:C1.+, CH3:R27.2
- removed net CH3:COLD_SEND: CH3:C3.+, CH3:R16.2, CH3:U1.10
- removed net CH3:HOT_IN: 3:IN.P$2, CH3:C2.+, CH3:R25.2
- removed net CH3:HOT_SEND: CH3:C5.+, CH3:R17.2, CH3:U1.12
- removed net CH3:N$1: CH3:C10.+, CH3:R13.2
- removed net CH3:N$11: CH3:C4.1, CH3:R19.1
- removed net CH3:N$12: CH3:C4.2, CH3:R20.1, CH3:R22.2, CH3:R26.1, CH3:U1.13
- removed net CH3:N$14: CH3:C1.-, CH3:C3.-, CH3:R23.2
- removed net CH3:N$15: CH3:C2.-, CH3:C5.-, CH3:R24.2
- removed net CH3:N$17: 3:GAIN.P$2, CH3:R26.2
- removed net CH3:N$2: CH3:C12.+, CH3:R15.2
- removed net CH3:N$23: CH3:C6.-, CH3:C7.-, CH3:R8.2
- removed net CH3:N$24: CH3:C11.1, CH3:U1.11
- removed net CH3:N$25: 3:U2.P$1, CH3:C6.+
- removed net CH3:N$26: CH3:C8.-, CH3:C9.-, CH3:R9.2
- removed net CH3:N$27: 3:U2.P$2, CH3:C8.+
- removed net CH3:N$28: CH3:C9.+, CH3:R10.2, CH3:R12.2
- removed net CH3:N$29: 3:GAIN1.A, CH3:C17.2, CH3:R11.2, CH3:U1.2
- removed net CH3:N$30: 3:GAIN2.A, CH3:C19.2, CH3:R14.2, CH3:U1.6
- removed net CH3:N$31: 3:GAIN1.E, 3:GAIN1.S, CH3:R13.1
- removed net CH3:N$33: CH3:R12.1, CH3:U1.3
- removed net CH3:N$34: 3:GAIN2.E, 3:GAIN2.S, CH3:R15.1
- removed net CH3:N$36: CH3:R18.1, CH3:U1.5
- removed net CH3:N$37: 3:BLEND.P$8, CH3:C19.1, CH3:R14.1, CH3:U1.7
- removed net CH3:N$9: 3:GAIN.P$3, CH3:R19.2, CH3:R20.2, CH3:R21.1, CH3:U1.8, CH3:U1.9
- removed net CH3:SND_RET_OUT: 3:BLEND.P$1, CH3:C17.1, CH3:R11.1, CH3:U1.1
- removed net N$61: C35.2, GAIN3.A, R55.2, U7.2
- new net 1:COLD_IN: 1:C1.+, 1:IN.P$3, 1:R27.2
- new net 1:COLD_SEND: 1:C3.+, 1:R16.2, 1:U1.10
- new net 1:HOT_IN: 1:C2.+, 1:IN.P$2, 1:R25.2
- new net 1:HOT_SEND: 1:C5.+, 1:R17.2, 1:U1.12
- new net 1:N$1: 1:C10.+, 1:R13.2
- new net 1:N$11: 1:C4.1, 1:R19.1
- new net 1:N$12: 1:C4.2, 1:R20.1, 1:R22.2, 1:R26.1, 1:U1.13
- new net 1:N$14: 1:C1.-, 1:C3.-, 1:R23.2
- new net 1:N$15: 1:C2.-, 1:C5.-, 1:R24.2
- new net 1:N$17: 1:GAIN.P$2, 1:R26.2
- new net 1:N$2: 1:C12.+, 1:R15.2
- new net 1:N$23: 1:C6.-, 1:C7.-, 1:R8.2
- new net 1:N$24: 1:C11.1, 1:U1.11
- new net 1:N$25: 1:C6.+, 1:U2.P$3
- new net 1:N$26: 1:C8.-, 1:C9.-, 1:R9.2
- new net 1:N$27: 1:C8.+, 1:U2.P$2
- new net 1:N$28: 1:C9.+, 1:R10.2, 1:R12.2
- new net 1:N$29: 1:C17.2, 1:GAIN1.E, 1:R11.2, 1:U1.2
- new net 1:N$3: 1:GAIN1.A, 1:GAIN1.S, 1:R13.1
- new net 1:N$30: 1:C19.2, 1:GAIN2.E, 1:R14.2, 1:U1.6
- new net 1:N$33: 1:R12.1, 1:U1.3
- new net 1:N$36: 1:R18.1, 1:U1.5
- new net 1:N$37: 1:BLEND.P$8, 1:C19.1, 1:R14.1, 1:U1.7
- new net 1:N$4: 1:GAIN2.A, 1:GAIN2.S, 1:R15.1
- new net 1:N$9: 1:GAIN.P$3, 1:R19.2, 1:R20.2, 1:R21.1, 1:U1.8, 1:U1.9
- new net 1:SND_RET_OUT: 1:BLEND.P$1, 1:C17.1, 1:R11.1, 1:U1.1
- new net 2:COLD_IN: 2:C1.+, 2:IN.P$3, 2:R27.2
- new net 2:COLD_SEND: 2:C3.+, 2:R16.2, 2:U1.10
- new net 2:HOT_IN: 2:C2.+, 2:IN.P$2, 2:R25.2
- new net 2:HOT_SEND: 2:C5.+, 2:R17.2, 2:U1.12
- new net 2:N$1: 2:C10.+, 2:R13.2
- new net 2:N$11: 2:C4.1, 2:R19.1
- new net 2:N$12: 2:C4.2, 2:R20.1, 2:R22.2, 2:R26.1, 2:U1.13
- new net 2:N$14: 2:C1.-, 2:C3.-, 2:R23.2
- new net 2:N$15: 2:C2.-, 2:C5.-, 2:R24.2
- new net 2:N$17: 2:GAIN.P$2, 2:R26.2
- new net 2:N$2: 2:C12.+, 2:R15.2
- new net 2:N$23: 2:C6.-, 2:C7.-, 2:R8.2
- new net 2:N$24: 2:C11.1, 2:U1.11
- new net 2:N$25: 2:C6.+, 2:U2.P$3
- new net 2:N$26: 2:C8.-, 2:C9.-, 2:R9.2
- new net 2:N$27: 2:C8.+, 2:U2.P$2
- new net 2:N$28: 2:C9.+, 2:R10.2, 2:R12.2
- new net 2:N$29: 2:C17.2, 2:GAIN1.E, 2:R11.2, 2:U1.2
- new net 2:N$3: 2:GAIN1.A, 2:GAIN1.S, 2:R13.1
- new net 2:N$30: 2:C19.2, 2:GAIN2.E, 2:R14.2, 2:U1.6
- new net 2:N$33: 2:R12.1, 2:U1.3
- new net 2:N$36: 2:R18.1, 2:U1.5
- new net 2:N$37: 2:BLEND.P$8, 2:C19.1, 2:R14.1, 2:U1.7
- new net 2:N$4: 2:GAIN2.A, 2:GAIN2.S, 2:R15.1
- new net 2:N$9: 2:GAIN.P$3, 2:R19.2, 2:R20.2, 2:R21.1, 2:U1.8, 2:U1.9
- new net 2:SND_RET_OUT: 2:BLEND.P$1, 2:C17.1, 2:R11.1, 2:U1.1
- new net 3:COLD_IN: 3:C1.+, 3:IN.P$3, 3:R27.2
- new net 3:COLD_SEND: 3:C3.+, 3:R16.2, 3:U1.10
- new net 3:HOT_IN: 3:C2.+, 3:IN.P$2, 3:R25.2
- new net 3:HOT_SEND: 3:C5.+, 3:R17.2, 3:U1.12
- new net 3:N$1: 3:C10.+, 3:R13.2
- new net 3:N$11: 3:C4.1, 3:R19.1
- new net 3:N$12: 3:C4.2, 3:R20.1, 3:R22.2, 3:R26.1, 3:U1.13
- new net 3:N$14: 3:C1.-, 3:C3.-, 3:R23.2
- new net 3:N$15: 3:C2.-, 3:C5.-, 3:R24.2
- new net 3:N$17: 3:GAIN.P$2, 3:R26.2
- new net 3:N$2: 3:C12.+, 3:R15.2
- new net 3:N$23: 3:C6.-, 3:C7.-, 3:R8.2
- new net 3:N$24: 3:C11.1, 3:U1.11
- new net 3:N$25: 3:C6.+, 3:U2.P$3
- new net 3:N$26: 3:C8.-, 3:C9.-, 3:R9.2
- new net 3:N$27: 3:C8.+, 3:U2.P$2
- new net 3:N$28: 3:C9.+, 3:R10.2, 3:R12.2
- new net 3:N$29: 3:C17.2, 3:GAIN1.E, 3:R11.2, 3:U1.2
- new net 3:N$3: 3:GAIN1.A, 3:GAIN1.S, 3:R13.1
- new net 3:N$30: 3:C19.2, 3:GAIN2.E, 3:R14.2, 3:U1.6
- new net 3:N$33: 3:R12.1, 3:U1.3
- new net 3:N$36: 3:R18.1, 3:U1.5
- new net 3:N$37: 3:BLEND.P$8, 3:C19.1, 3:R14.1, 3:U1.7
- new net 3:N$4: 3:GAIN2.A, 3:GAIN2.S, 3:R15.1
- new net 3:N$9: 3:GAIN.P$3, 3:R19.2, 3:R20.2, 3:R21.1, 3:U1.8, 3:U1.9
- new net 3:SND_RET_OUT: 3:BLEND.P$1, 3:C17.1, 3:R11.1, 3:U1.1
- net +48V: now also 1:R25.1, 1:R27.1, 2:R25.1, 2:R27.1, 3:R25.1, 3:R27.1; no longer CH1:R25.1, CH1:R27.1, CH2:R25.1, CH2:R27.1, CH3:R25.1, CH3:R27.1
- net +9V: now also 1:C11.2, 1:U1.4, 2:C11.2, 2:U1.4, 3:C11.2, 3:U1.4, R65.1; no longer BYPASS.P$1, CH1:C11.2, CH1:U1.4, CH2:C11.2, CH2:U1.4, CH3:C11.2, CH3:U1.4
- net DRY1: now also 1:C7.+, 1:R18.2, 1:R22.1, 1:U1.14; no longer CH1:C7.+, CH1:R18.2, CH1:R22.1, CH1:U1.14
- net DRY2: now also 2:C7.+, 2:R18.2, 2:R22.1, 2:U1.14; no longer CH2:C7.+, CH2:R18.2, CH2:R22.1, CH2:U1.14
- net DRY3: now also 3:C7.+, 3:R18.2, 3:R22.1, 3:U1.14; no longer CH3:C7.+, CH3:R18.2, CH3:R22.1, CH3:U1.14
- net GND: now also 1:C10.-, 1:C12.-, 1:R23.1, 1:R24.1, 1:R8.1, 1:R9.1, 1:U2.P$1, 2:C10.-, 2:C12.-, 2:R23.1, 2:R24.1, 2:R8.1, 2:R9.1, 2:U2.P$1, 3:C10.-, 3:C12.-, 3:R23.1, 3:R24.1, 3:R8.1, 3:R9.1, 3:U2.P$1, LOOPMASTER.P$1, U$2.GND; no longer 1:U2.P$3, 2:U2.P$3, 3:U2.P$3, CH1:C10.-, CH1:C12.-, CH1:R23.1, CH1:R24.1, CH1:R8.1, CH1:R9.1, CH2:C10.-, CH2:C12.-, CH2:R23.1, CH2:R24.1, CH2:R8.1, CH2:R9.1, CH3:C10.-, CH3:C12.-, CH3:R23.1, CH3:R24.1, CH3:R8.1, CH3:R9.1, LOOPMASTER.P$3, R65.1
- net MIX_OUT: now also C14.-, R8.2
- net N$23: now also GAIN1.A, GAIN1.S, R13.1; no longer C14.-, R8.2
- net N$29: now also GAIN1.E; no longer GAIN1.A
- net N$30: now also GAIN2.E; no longer GAIN2.A
- net N$31: now also GAIN2.A, GAIN2.S, R15.1; no longer GAIN1.E, GAIN1.S, R13.1
- net N$34: now also GAIN4.A, GAIN4.S, R62.1; no longer GAIN2.E, GAIN2.S, R15.1
- net N$62: now also GAIN3.A; no longer GAIN3.E
- net N$66: now also GAIN4.E; no longer GAIN4.A
- net N$67: now also C35.2, GAIN3.E, R55.2, U7.2; no longer GAIN4.E, GAIN4.S, R62.1
- net SELECT: now also U$2.HOT
- net SND: now also LOOPMASTER.P$3; no longer LOOPMASTER.P$1
- net VDD: now also 1:R10.1, 1:R16.1, 1:R17.1, 1:R21.2, 2:R10.1, 2:R16.1, 2:R17.1, 2:R21.2, 3:R10.1, 3:R16.1, 3:R17.1, 3:R21.2; no longer CH1:R10.1, CH1:R16.1, CH1:R17.1, CH1:R21.2, CH2:R10.1, CH2:R16.1, CH2:R17.1, CH2:R21.2, CH3:R10.1, CH3:R16.1, CH3:R17.1, CH3:R21.2
