File: mixer.sch (EAGLE design)
At the start: 133 parts, among them U1 TL074IDT, U2 TL074IDT, U3 TL074IDT, U4 TL074IDT, U5 TL074IDT, U6 TL074IDT, U7 TL074IDT

Commit message: Started board layout and removed EQ
Parts:
- removed C39: 10u, 16V, passives:C-PR-SMD-SV-A
- removed C40, C41, C42: 100 n, passives:C-EUC0603
- removed GAIN: 10 k, passives:RK09L1140
- removed TC, TC1, TC2, TC3: HOT_COLD, connectors:HOT_COLD
- removed U$2: SEND_RETURN, connectors:SEND_RETURN
- removed U$3, U$4: LEFT_RIGHT, connectors:LEFT_RIGHT
- added BYPASS, MONO: BUTTON, connectors:BUTTON
- added D1, D2: 1N4004, passives:1N4004
- added GAIN5: 10 k, passives:TRIM_EU-RJ9W
- added LD1: (no value), passives:DUOLED-RG-A
- added LOOPMASTER: SEND_RETURN, connectors:SEND_RETURN
- added MON_IN, MON_THROUGH, OUT_L, OUT_R, TC_SEND_JACK: HOT_COLD, connectors:HOT_COLD
- added MON_OUT: LEFT_RIGHT, connectors:LEFT_RIGHT
- added R64, R65: 10 k, passives:R-EU_0204/7
- added TC_RET: LEFT_RIGHT_BYPASS, connectors:LEFT_RIGHT_BYPASS
- added U$10: SBC1-102-211, passives:SBC1-102-211
- added U$5: ADG333ABNZADG333ABNZ, ic:ADG333ABNZADG333ABNZ
- added U$6: ADG436BNZADG436BNZ, ic:ADG436BNZADG436BNZ
- added U8: TL074, ic:TL074IDTPDIP-14
- added U9: V7809W-500R, power:V7809W-500R
- C1, C10, C13, C14, C15, C16, C18, C2, C20, C22, C3, C36, C4, C5, C8, C9: value 10u, 16V -> 10u; device passives:C-PR-SMD-SV-A -> passives:C-PR-2,0X5; LINK https://www.mouser.se/ProductDetail/Nichicon/UWX1C100MCL2GB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 -> (none); MFR Nichicon -> (none); MFR-NR UWX1C100MCL2GB -> (none); SUPPLIER Mouser -> (none)
- C11, C26: value 100 n -> 10u; device passives:C-EUC0603 -> passives:C-PR-2,0X5
- C12, C21, C24, C25, C32, C6, C7: value 33u, 63V -> 10u, 63V; device passives:C-PR-SMD-SV-E/F -> passives:C-PR-2,0X6; LINK https://www.mouser.se/ProductDetail/Panasonic/EEE-FK1J330P?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 -> (none); MFR Panasonic -> (none); MFR-NR EEE-FK1J330P -> (none); SUPPLIER Mouser -> (none)
- C17, C19, C28, C29, C34, C35, C37, C38: device passives:C-EUC0603 -> passives:C-EU025-025X050
- C23: value 10u, 16V -> 10u, 63V; device passives:C-PR-SMD-SV-A -> passives:C-PR-2,0X6; LINK https://www.mouser.se/ProductDetail/Nichicon/UWX1C100MCL2GB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 -> (none); MFR Nichicon -> (none); MFR-NR UWX1C100MCL2GB -> (none); SUPPLIER Mouser -> (none)
- C27: value 100 n -> 2.2u, 63V; device passives:C-EUC0603 -> passives:C-PR-2,0X6
- C30: value 10u, 16V -> 2.2u, 63V; device passives:C-PR-SMD-SV-A -> passives:C-PR-2,0X6; LINK https://www.mouser.se/ProductDetail/Nichicon/UWX1C100MCL2GB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 -> (none); MFR Nichicon -> (none); MFR-NR UWX1C100MCL2GB -> (none); SUPPLIER Mouser -> (none)
- C31: value 10u, 16V -> 390 u / 63 V; device passives:C-PR-SMD-SV-A -> passives:C-PR-5,0X12,5; LINK https://www.mouser.se/ProductDetail/Nichicon/UWX1C100MCL2GB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 -> (none); MFR Nichicon -> (none); MFR-NR UWX1C100MCL2GB -> (none); SUPPLIER Mouser -> (none)
- C33: value 33u, 63V -> 10u; device passives:C-PR-SMD-SV-E/F -> passives:C-PR-2,0X5; LINK https://www.mouser.se/ProductDetail/Panasonic/EEE-FK1J330P?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 -> (none); MFR Panasonic -> (none); MFR-NR EEE-FK1J330P -> (none); SUPPLIER Mouser -> (none)
- GAIN1, GAIN2, GAIN3, GAIN4: device passives:TRIM_EU-ECP10P -> passives:TRIM_EU-RJ9W
- R1, R10, R11, R12, R13, R14, R15, R16, R17, R18, R19, R2, R20, R21, R22, R23, R24, R25, R26, R27, R28, R29, R3, R30, R31, R32, R33, R34, R35, R36, R37, R38, R39, R4, R40, R41, R42, R43, R44, R45, R46, R47, R48, R49, R5, R50, R51, R52, R53, R54, R55, R56, R57, R58, R59, R6, R60, R61, R62, R63, R7, R8, R9: device passives:R-EU_R0603 -> passives:R-EU_0204/7
- U$1: value UTBULT_DESIGN4 -> UTBULT_DESIGN3; device misc:UTBULT_DESIGN4 -> misc:UTBULT_DESIGN3
- U1, U2, U3, U4, U5, U6, U7: value TL074IDT -> TL074; device ic:TL074IDT -> ic:TL074IDTPDIP-14
Connections:
- removed net EQ_IN: C12.-, R5.1, U2G$1.IN+
- removed net OUT_MIX: U$2.2
- removed net RET_L: VOLUME1G$1.3
- removed net RET_R: VOLUME1G$2.3
- removed net SEL_OUT: U$2.3
- removed net SEL_WET: BLEND1G$1.2, BLEND1G$2.2
- removed net TC_DRY: BLEND1G$1.2, BLEND1G$2.2, R3.2, R6.2
- new net MASTER_MON_L: U$6.D2, VOLUM6G$1.3, VOLUME1G$2.3
- new net MASTER_MON_R: U$6.D1, VOLUM6G$2.3, VOLUME1G$1.3
- new net N$65: U$6.S1B, U8G$1.IN-, U8G$1.OUT
- new net N$70: D1.A, U9.VO_P
- new net N$71: U$6.S2B, U8G$2.IN-, U8G$2.OUT
- new net N$72: MONO.P$3, VOLUM6G$2.2
- new net N$73: C28.1, R45.2, R46.1, U7G$4.IN+
- new net N$74: LD1.CR, U$5.S4B
- new net N$75: LD1.CG, U$5.S4A
- new net N$76: R64.1, U$5.D4
- new net N$79: C27.+, U$10.P$1, U9.VIN_P
- new net N$81: D2.A, PWR$1.VCC
- new net RET1: U$5.D1
- new net RET2: U$5.D2
- new net RET3: U$5.D3
- new net SELECT: BYPASS.P$2, R65.2, U$5.IN1, U$5.IN2, U$5.IN3, U$5.IN4, U$6.IN1, U$6.IN2
- new net TC_BALANCED: BLEND1G$1.2, BLEND1G$2.2, R3.2, R6.2, U8G$3.IN+, U8G$4.IN+
- new net TC_BYPASS_L: TC_RET.BYPASS_LEFT, U8G$3.IN-, U8G$3.OUT
- new net TC_BYPASS_R: TC_RET.BYPASS_RIGHT, U8G$4.IN-, U8G$4.OUT
- new net WET1: U$5.S1A
- new net WET2: U$5.S2A
- new net WET3: U$5.S3A
- net +48V: now also C30.+, C31.+, U$10.P$2
- net +9V: now also BYPASS.P$1, D1.C, D2.C, R64.2, U$5.VDD, U$6.VDD, U8G$5.V+; no longer C10.2, C11.1, C26.1, C27.1, C37.1, C40.1, C41.1, C42.1, PWR$1.VCC
- net COLD_IN: now also C1.+; no longer C7.+, TC.COLD
- net COLD_SEND: now also C11.+, C3.+; no longer C30.+, C8.+
- net DRY1: now also U$5.S1B
- net DRY2: now also U$5.S2B
- net DRY3: now also U$5.S3B
- net GND: now also BYPASS.P$3, C10.-, C12.-, C27.-, C30.-, C31.-, C33.-, LD1.A, LOOPMASTER.GND, MON_IN.GND, MON_OUT.GND, MON_THROUGH.GND, OUT_L.GND, OUT_R.GND, R65.1, TC_RET.GND, TC_SEND_JACK.GND, U$5.GND, U$5.VSS, U$6.GND, U$6.VSS, U2G$1.GND, U8G$5.V-, U9.GND; no longer C11.2, C26.2, C27.2, C39.-, C40.2, C41.2, C42.2, GAIN.P$1, R5.2, TC.GND, TC1.GND, TC2.GND, TC3.GND, U$1.GND, U$2.GND, U$2.P$1, U$3.GND, U$4.GND
- net HOT_IN: now also C2.+; no longer C6.+, TC.HOT
- net HOT_SEND: now also C26.+, C5.+; no longer C31.+, C9.+
- net L_COLD: now also OUT_L.COLD; no longer TC1.COLD
- net L_HOT: now also OUT_L.HOT; no longer TC1.HOT
- net MIX_OUT: now also R18.2, U8G$1.IN+, U8G$2.IN+
- net MON_COLD: now also C25.+, MON_IN.COLD, MON_THROUGH.COLD; no longer C33.+, TC3.COLD
- net MON_HOT: now also MON_IN.HOT, MON_THROUGH.HOT; no longer TC3.HOT
- net MON_OUT_L: now also MON_OUT.LEFT; no longer U$4.LEFT
- net MON_OUT_R: now also MON_OUT.RIGHT; no longer U$4.RIGHT
- net N$1: now also C10.+, R13.2; no longer R1.2, U2G$1.IN-, U2G$1.OUT
- net N$10: no longer R3.2
- net N$12: now also C2.-; no longer C3.-
- net N$13: no longer C12.+, R22.1, U1G$4.OUT
- net N$14: now also C1.-, C3.-, C6.-; no longer C7.-
- net N$15: now also C2.-, C5.-, C7.-; no longer C6.-
- net N$16: no longer C3.1
- net N$17: no longer GAIN.2
- net N$18: no longer C5.2, R4.2
- net N$19: no longer C3.2
- net N$2: now also C12.+, R15.2; no longer R1.1, U2G$4.IN+
- net N$20: no longer R4.1, U2G$3.IN-, U2G$3.OUT
- net N$21: no longer C5.1, R6.1, U2G$3.IN+
- net N$22: no longer R6.2
- net N$23: now also C6.-, C7.-; no longer C13.-
- net N$24: no longer C10.1, U2G$5.V-
- net N$25: now also C11.-, C25.-, C6.+, U2G$1.SEND; no longer C14.+, C30.-, C33.-, U$1.SEND
- net N$26: now also C8.-, C9.-
- net N$27: now also C26.-, C8.+, U2G$1.RETURN; no longer C15.+, C31.-, U$1.RETURN
- net N$28: now also C9.+
- net N$3: no longer C1.2
- net N$4: no longer R7.2, U2G$4.IN-
- net N$42: now also C13.-, C23.-; no longer C22.-, C25.-
- net N$43: now also C22.-; no longer C23.-
- net N$44: now also C13.+; no longer C22.+
- net N$45: now also C22.+; no longer C23.+
- net N$46: now also GAIN5.E; no longer GAIN.3
- net N$5: no longer C1.1
- net N$50: now also GAIN5.S; no longer GAIN.2
- net N$51: now also MONO.P$1
- net N$58: now also MONO.P$2; no longer VOLUM6G$2.2
- net N$6: no longer C2.2, R2.2
- net N$63: now also C33.+; no longer C36.+
- net N$68: now also C36.+; no longer C39.+
- net N$7: no longer R2.1, U2G$2.IN-, U2G$2.OUT
- net N$8: no longer C2.1, R3.1, U2G$2.IN+
- net N$9: now also C3.-; no longer C2.-, GAIN.3
- net OUT_L: now also VOLUME1G$2.2; no longer VOLUME1G$1.2
- net OUT_R: now also VOLUME1G$1.2; no longer VOLUME1G$2.2
- net RET: now also LOOPMASTER.RETURN; no longer U$2.RETURN
- net R_COLD: now also OUT_R.COLD; no longer TC2.COLD
- net R_HOT: now also C23.+, OUT_R.HOT; no longer C25.+, TC2.HOT
- net SEL_DRY: now also C7.+, R22.1, U1G$4.OUT; no longer C13.+, R7.1, U2G$4.OUT
- net SND: now also LOOPMASTER.SEND; no longer U$2.SEND
- net TC_COLD: now also C7.+, TC_SEND_JACK.COLD; no longer C6.+, TC.COLD
- net TC_HOT: now also C6.+, TC_SEND_JACK.HOT; no longer C7.+, TC.HOT
- net TC_RET_L: now also TC_RET.LEFT; no longer U$3.LEFT
- net TC_RET_R: now also C2.+, TC_RET.RIGHT; no longer C3.+, U$3.RIGHT
- net TC_WET_L: now also C3.+, U$6.S1A; no longer C2.+, VOLUM6G$1.3
- net TC_WET_R: now also U$6.S2A; no longer VOLUM6G$2.3
- net VDD: now also C37.1, U7G$4.IN-, U7G$4.OUT; no longer C28.1, R45.2, R46.1, U$2.1
Other:
- note added: "Comes from BLEND_SEL_VOL"
- note added: "Comes from MIXER"
- note added: "Comes from TC_RET jack"
- note added: "Goes to L_OUT jack"
- note added: "Goes to MON_MIX"
- note added: "Goes to R_OUT jack"
- note added: "Goes to SND_RET_JACK"
- note added: "Goes to TC_RET_SEL, SND_RET and BLEND_SEL_VOL"
- note added: "Goes to TC_SEND and TC_RETURN"
- note added: "Goes to TC_SEND jack"
- moved on the sheet: BLEND1G$1, BLEND1G$2, C1, C10, C12, C13, C14, C15, C16, C17, C18, C19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

Commit message: Swapped gain trimpots and started restructuring
Parts:
- added U$2: UNBALANCED_INPUT_JACK, connectors:UNBALANCED_INPUT_JACK
Connections:
- removed net N$61: C35.2, GAIN3.A, R55.2, U7G$1.IN-
- net +9V: now also R65.1; no longer BYPASS.P$1
- net GND: now also U$2.GND; no longer R65.1
- net MIX_OUT: now also C14.-, R8.2
- net N$23: now also GAIN1.A, GAIN1.S, R13.1; no longer C14.-
- net N$29: now also GAIN1.E; no longer GAIN1.A
- net N$3: now also GAIN1.A, GAIN1.S, R13.1
- net N$30: now also GAIN2.E; no longer GAIN2.A
- net N$31: now also GAIN2.A, GAIN2.S, R15.1; no longer GAIN1.E, GAIN1.S, R13.1
- net N$34: now also GAIN4.A, GAIN4.S, R62.1; no longer GAIN2.E, GAIN2.S, R15.1
- net N$4: now also GAIN2.A, GAIN2.S, R15.1
- net N$62: now also GAIN3.A; no longer GAIN3.E
- net N$66: now also GAIN4.E; no longer GAIN4.A
- net N$67: now also C35.2, GAIN3.E, R55.2, U7G$1.IN-; no longer GAIN4.E, GAIN4.S, R62.1
- net SELECT: now also U$2.HOT
Other:
- moved on the sheet: BLEND1G$1, BLEND1G$2, C19, C20, GAIN1, GAIN2, GAIN3, GAIN4, R14, R15, R18, U2G$2
